File: hardware/motor_pcb/_autosave-motor_pcb.kicad_sch (KiCad schematic)
At the start: 23 parts, among them J1 Conn_01x14, J2 Conn_01x03, J3 Conn_01x14, U1 TMC6300, U2 MT6701-CT

Commit message: Routed motor pcb
Parts:
- gave numbers to parts that had none: 1
Changed lines of the file:
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@@
   (symbol (lib_id "Device:C") (at 181.61 81.28 0) (unit 1)
     (in_bom yes) (on_board yes) (fields_autoplaced)
-    (property "Reference" "C?" (id 0) (at 185.42 80.0099 0)
+    (property "Reference" "C6" (id 0) (at 185.42 80.0099 0)
       (effects (font (size 1.27 1.27)) (justify left))
     )
@@
     )
     (path "/ced9211e-3830-49a7-9c5a-53307e7d1f43"
-      (reference "C?") (unit 1) (value "100nF") (footprint "Capacitor_SMD:C_0603_1608Metric")
+      (reference "C6") (unit 1) (value "100nF") (footprint "Capacitor_SMD:C_0603_1608Metric")
     )
     (path "/27b1ed45-aefd-4e31-91ba-488f859fc1d8"
