File: hardware/motor_pcb/motor_pcb.kicad_pcb (KiCad board)
At the start: 4 copper layers, 36 x 36 mm, 23 parts, among them J1 Conn_01x14, J2 Conn_01x03, J3 Conn_01x14, U1 TMC6300, U2 MT6701-CT

Commit message: Fixed routing
Parts:
- moved J1 23.1 mm to (38.5, 38.6), turned to 45 degrees
- moved J3 22.9 mm to (61.3, 38.5), turned to -45 degrees
- moved C1 17.1 mm to (64.4, 56.2)
- moved C4 15.1 mm to (60.5, 58.5), turned to 180 degrees
- moved U1 11.0 mm to (55.0, 59.3), turned to -135 degrees
- moved C5 9.86 mm to (49.6, 58.8)
- moved C6 9.47 mm to (54.1, 65.8)
- moved R1 8.78 mm to (61.2, 60.5), turned to 0 degrees
- moved C2 8.61 mm to (56.5, 64.2)
Connections:
- J1 pad 1: +5V -> GND
- J1 pad 11: GND -> +5V
- J1 pad 12: GND -> +5V
- J1 pad 13: GND -> +5V
- J1 pad 14: GND -> +5V
- J1 pad 2: +5V -> GND
- J1 pad 3: +5V -> GND
- J1 pad 4: +5V -> GND
- J3 pad 1: +3V3 -> GND
- J3 pad 10: /SDA -> /DIAG
- J3 pad 11: /SCL -> /SDA
- J3 pad 12: GND -> /SCL
- J3 pad 13: GND -> +3V3
- J3 pad 14: GND -> +3V3
- J3 pad 2: +3V3 -> GND
- J3 pad 3: /VL -> GND
- J3 pad 4: /WL -> /VL
- J3 pad 5: /UL -> /WL
- J3 pad 6: /WH -> /UL
- J3 pad 7: /VH -> /WH
- J3 pad 8: /UH -> /VH
- J3 pad 9: /DIAG -> /UH
- U1 pad 1: Net-(J2-Pad3) -> Net-(J2-Pad1)
- U1 pad 15: Net-(J2-Pad1) -> Net-(J2-Pad3)
Routing:
- net Net-(J1-Pad9): track 49.8 -> 29.6 mm
- net Net-(J1-Pad5): track 34.3 -> 15.5 mm
- net Net-(J1-Pad6): track 38.2 -> 19.9 mm
- net Net-(J1-Pad7): track 41.3 -> 23.4 mm
- net Net-(J1-Pad8): track 45.5 -> 27.9 mm
- net Net-(J2-Pad1): track 17.0 -> 3.97 mm
- net /SCL: track 17.0 -> 28.5 mm, vias 0 -> 2
- net Net-(J2-Pad3): track 14.7 -> 3.50 mm
- net Net-(J1-Pad10): track 45.0 -> 33.9 mm
- net Net-(J2-Pad2): track 12.1 -> 3.50 mm
- net /SDA: track 19.6 -> 27.4 mm
- net +5V: track 7.55 -> 12.1 mm, vias 11 -> 10
- net Net-(R1-Pad1): track 14.2 -> 17.9 mm
- net Net-(C6-Pad1): track 2.42 -> 5.74 mm
- net /UL: track 26.5 -> 24.1 mm
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