File: hardware/motor_pcb/motor_pcb.kicad_sch (KiCad schematic)
At the start: 23 parts, among them J1 Conn_01x14, J2 Conn_01x03, J3 Conn_01x14, U1 TMC6300, U2 MT6701-CT

Commit message: Fixed routing
Parts:
- C1: LCSC (none) -> C45783
- C2, C3, C4, C5, C6: LCSC (none) -> C14663
- R1: LCSC (none) -> C37936
- R2, R3: LCSC (none) -> C23162
- U2: LCSC (none) -> C2856764
Connections:
- net +3V3: now also J3.13 (Pin_13), J3.14 (Pin_14); no longer J3.1 (Pin_1), J3.2 (Pin_2)
- net +5V: now also J1.11 (Pin_11), J1.12 (Pin_12), J1.13 (Pin_13), J1.14 (Pin_14); no longer J1.1 (Pin_1), J1.2 (Pin_2), J1.3 (Pin_3), J1.4 (Pin_4)
- net DIAG: now also J3.10 (Pin_10); no longer J3.9 (Pin_9)
- net GND: now also J1.1 (Pin_1), J1.2 (Pin_2), J1.3 (Pin_3), J1.4 (Pin_4), J3.1 (Pin_1), J3.2 (Pin_2), J3.3 (Pin_3); no longer J1.11 (Pin_11), J1.12 (Pin_12), J1.13 (Pin_13), J1.14 (Pin_14), J3.12 (Pin_12), J3.13 (Pin_13), J3.14 (Pin_14)
- net SCL: now also J3.12 (Pin_12); no longer J3.11 (Pin_11)
- net SDA: now also J3.11 (Pin_11); no longer J3.10 (Pin_10)
- net UH: now also J3.9 (Pin_9); no longer J3.8 (Pin_8)
- net UL: now also J3.6 (Pin_6); no longer J3.5 (Pin_5)
- net VH: now also J3.8 (Pin_8); no longer J3.7 (Pin_7)
- net VL: now also J3.4 (Pin_4); no longer J3.3 (Pin_3)
- net WH: now also J3.7 (Pin_7); no longer J3.6 (Pin_6)
- net WL: now also J3.5 (Pin_5); no longer J3.4 (Pin_4)
- net at J2.1 (Pin_1): now also U1.1 (W); no longer U1.15 (U)
- net at J2.3 (Pin_3): now also U1.15 (U); no longer U1.1 (W)
Other:
- moved on the sheet: J1, J3, TP2, TP3, TP4, TP5, TP6, TP7
