File: hardware/main_pcb/main_pcb.kicad_pcb (KiCad board)
At the start: 2 copper layers, 44.5 x 44.5 mm, 58 parts, among them J1 USB_C_Receptacle_USB2.0, J2 BAT, J3 PWR, J4 MOTOR, J5 LCD, J6 PROG, Q1 AO3400A, Q2 AO3400A, Q3 AO3400A, SW1 SW_SPST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

Commit message: Switch to 4 layer pcb
Other:
- copper layers 2 -> 4
Changed lines of the file:
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@@
 (kicad_pcb (version 20211014) (generator pcbnew)
   (general
-    (thickness 1.6)
+    (thickness 4.69)
   )
   (paper "A4")
   (layers
     (0 "F.Cu" signal)
+    (1 "In1.Cu" signal)
+    (2 "In2.Cu" signal)
     (31 "B.Cu" signal)
     (32 "B.Adhes" user "B.Adhesive")
@@
   )
   (setup
+    (stackup
+      (layer "F.SilkS" (type "Top Silk Screen"))
+      (layer "F.Paste" (type "Top Solder Paste"))
+      (layer "F.Mask" (type "Top Solder Mask") (thickness 0.01))
+      (layer "F.Cu" (type "copper") (thickness 0.035))
+      (layer "dielectric 1" (type "core") (thickness 1.51) (material "FR4") (epsilon_r 4.5) (loss_tangent 0.02))
+      (layer "In1.Cu" (type "copper") (thickness 0.035))
+      (layer "dielectric 2" (type "prepreg") (thickness 1.51) (material "FR4") (epsilon_r 4.5) (loss_tangent 0.02))
+      (layer "In2.Cu" (type "copper") (thickness 0.035))
+      (layer "dielectric 3" (type "core") (thickness 1.51) (material "FR4") (epsilon_r 4.5) (loss_tangent 0.02))
+      (layer "B.Cu" (type "copper") (thickness 0.035))
+      (layer "B.Mask" (type "Bottom Solder Mask") (thickness 0.01))
+      (layer "B.Paste" (type "Bottom Solder Paste"))
+      (layer "B.SilkS" (type "Bottom Silk Screen"))
+      (copper_finish "None")
+      (dielectric_constraints no)
+    )
     (pad_to_mask_clearance 0)
     (pcbplotparams

Commit message: Updated connectors
Parts:
- removed J5: LCD, Connector_Hirose:Hirose_DF52-8S-0.8H_1x08-1MP_P0.80mm_Horizontal
- D1, D2, D3, D4, D5, D6, D7, D8: moved to B.Cu
- J3: value PWR -> Conn_01x14; footprint Connector_PinSocket_2.54mm:PinSocket_1x02_P2.54mm_Vertical -> Jushuo:FPC_14; moved to B.Cu
- J4: value MOTOR -> Conn_01x14; footprint Connector_Hirose:Hirose_DF52-12S-0.8H_1x12-1MP_P0.80mm_Horizontal -> Jushuo:FPC_14; moved to B.Cu
- moved D2 101.4 mm to (31.5, 42.4), turned to -112.5 degrees
- moved D1 97.8 mm to (42.4, 68.5), turned to -22.5 degrees
- moved J4 89.5 mm to (41.1, 41.1), turned to 45 degrees
- moved D5 82.8 mm to (31.5, 57.6), turned to -67.5 degrees
- moved D3 82.1 mm to (57.6, 31.5), turned to 157.5 degrees
- moved D6 77.8 mm to (42.4, 31.5), turned to 22.5 degrees
- moved D8 66.5 mm to (57.6, 68.5), turned to 22.5 degrees
- moved D4 60.7 mm to (68.5, 57.6), turned to 67.5 degrees
- moved D7 44.2 mm to (68.5, 42.4), turned to 112.5 degrees
- moved J3 13.9 mm to (58.9, 41.1), turned to -45 degrees
Connections:
- J3 pad 2: +5V -> GND
- J4 pad 1: +3.3V -> GND
- J4 pad 10: MM_SCL -> LCD_BL
- J4 pad 11: MM_CS -> +5V
- J4 pad 12: GND -> +5V
- J4 pad 2: MOTOR_UH -> GND
- J4 pad 3: MOTOR_UL -> GND
- J4 pad 4: MOTOR_VH -> GND
- J4 pad 5: MOTOR_VL -> LCD_RESET
- J4 pad 6: MOTOR_WH -> LCD_SDA
- J4 pad 7: MOTOR_WL -> LCD_SCL
- J4 pad 8: MOTOR_DIAG -> LCD_CS
- J4 pad 9: MM_SDA -> LCD_DC

Commit message: Updated battery connector
Parts:
- J2: value BAT -> Conn_01x03; footprint Connector_JST:JST_XH_B2B-XH-AM_1x02_P2.50mm_Vertical -> Connector_Molex:Molex_PicoBlade_53261-0371_1x03-1MP_P1.25mm_Horizontal
Connections:
- J2 pad 2: GND -> unconnected-(J2-Pad2)
Changed lines of the file:
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@@
   (net 91 "unconnected-(U4-Pad38)")
   (net 92 "unconnected-(U4-Pad39)")
+  (net 93 "unconnected-(J2-Pad2)")
   (footprint "Resistor_SMD:R_0603_1608Metric" (layer "F.Cu")
     (at 121.67 119.555)
@@
     )
   )
-  (footprint "Connector_JST:JST_XH_B2B-XH-AM_1x02_P2.50mm_Vertical" (layer "F.Cu")
+  (footprint "Connector_Molex:Molex_PicoBlade_53261-0371_1x03-1MP_P1.25mm_Horizontal" (layer "F.Cu")
     (at 126.34 90.075)
-    (descr "JST XH series connector, B2B-XH-AM, with boss (http://www.jst-mfg.com/product/pdf/eng/eXH.pdf), generated with kicad-footprint-generator")
-    (tags "connector JST XH vertical boss")
-    (property "Sheetfile" "main_pcb.kicad_sch")
-    (property "Sheetname" "")
-    (attr through_hole)
-    (fp_text reference "J2" (at 1.25 -3.55) (layer "F.SilkS")
-      (effects (font (size 1 1) (thickness 0.15)))
-    )
-    (fp_text value "BAT" (at 1.25 4.6) (layer "F.Fab")
-      (effects (font (size 1 1) (thickness 0.15)))
-    )
-    (fp_text user "${REFERENCE}" (at 1.25 2.7) (layer "F.Fab")
-      (effects (font (size 1 1) (thickness 0.15)))
-    )
-    (fp_line (start -0.75 -1.7) (end -0.75 -2.45) (layer "F.SilkS") (width 0.12))
-    (fp_line (start 4.3 -0.2) (end 4.3 2.75) (layer "F.SilkS") (width 0.12))
-    (fp_line (start -2.56 -2.46) (end -2.56 3.51) (layer "F.SilkS") (width 0.12))
-    (fp_line (start -2.85 -2.75) (end -2.85 -1.5) (layer "F.SilkS") (width 0.12))
-    (fp_line (start 5.05 -2.45) (end 3.25 -2.45) (layer "F.SilkS") (width 0.12))
-    (fp_line (start 4.3 2.75) (end 1.25 2.75) (layer "F.SilkS") (width 0.12))
-    (fp_line (start 0.75 -1.7) (end 1.75 -1.7) (layer "F.SilkS") (width 0.12))
-    (fp_line (start 0.75 -2.45) (end 0.75 -1.7) (layer "F.SilkS") (width 0.12))
-    (fp_line (start 1.75 -1.7) (end 1.75 -2.45) (layer "F.SilkS") (width 0.12))
-    (fp_line (start -2.55 -2.45) (end -2.55 -1.7) (layer "F.SilkS") (width 0.12))
-    (fp_line (start -2.55 -0.2) (end -1.8 -0.2) (layer "F.SilkS") (width 0.12))
-    (fp_line (start 3.25 -1.7) (end 5.05 -1.7) (layer "F.SilkS") (width 0.12))
-    (fp_line (start 1.75 -2.45) (end 0.75 -2.45) (layer "F.SilkS") (width 0.12))
-    (fp_line (start -1.8 -0.2) (end -1.8 1.14) (layer "F.SilkS") (width 0.12))
-    (fp_line (start -2.55 -1.7) (end -0.75 -1.7) (layer "F.SilkS") (width 0.12))
-    (fp_line (start -0.75 -2.45) (end -2.55 -2.45) (layer "F.SilkS") (width 0.12))
-    (fp_line (start 5.06 -2.46) (end -2.56 -2.46) (layer "F.SilkS") (width 0.12))
-    (fp_line (start 1.25 2.75) (end -0.74 2.75) (layer "F.SilkS") (width 0.12))
-    (fp_line (start -2.56 3.51) (end 5.06 3.51) (layer "F.SilkS") (width 0.12))
-    (fp_line (start -1.6 -2.75) (end -2.85 -2.75) (layer "F.SilkS") (width 0.12))
-    (fp_line (start 3.25 -2.45) (end 3.25 -1.7) (layer "F.SilkS") (width 0.12))
-    (fp_line (start 5.05 -0.2) (end 4.3 -0.2) (layer "F.SilkS") (width 0.12))
-    (fp_line (start 5.06 3.51) (end 5.06 -2.46) (layer "F.SilkS") (width 0.12))
-    (fp_line (start 5.05 -1.7) (end 5.05 -2.45) (layer "F.SilkS") (width 0.12))
-    (fp_line (start 5.45 3.9) (end 5.45 -2.85) (layer "F.CrtYd") (width 0.05))
-    (fp_line (start -2.95 -2.85) (end -2.95 3.9) (layer "F.CrtYd") (width 0.05))
-    (fp_line (start 5.45 -2.85) (end -2.95 -2.85) (layer "F.CrtYd") (width 0.05))
-    (fp_line (start -2.95 3.9) (end 5.45 3.9) (layer "F.CrtYd") (width 0.05))
-    (fp_line (start 4.95 3.4) (end 4.95 -2.35) (layer "F.Fab") (width 0.1))
-    (fp_line (start 0 -1.35) (end 0.625 -2.35) (layer "F.Fab") (width 0.1))
-    (fp_line (start 4.95 -2.35) (end -2.45 -2.35) (layer "F.Fab") (width 0.1))
-    (fp_line (start -0.625 -2.35) (end 0 -1.35) (layer "F.Fab") (width 0.1))
-    (fp_line (start -2.45 3.4) (end 4.95 3.4) (layer "F.Fab") (width 0.1))
-    (fp_line (start -2.45 -2.35) (end -2.45 3.4) (layer "F.Fab") (width 0.1))
-    (pad "" np_thru_hole circle (at -1.6 2) (size 1.2 1.2) (drill 1.2) (layers *.Cu *.Mask))
-    (pad "1" thru_hole roundrect (at 0 0) (size 1.7 2) (drill 1) (layers *.Cu *.Mask) (roundrect_rratio 0.147059)
+    (descr "Molex PicoBlade series connector, 53261-0371 (http://www.molex.com/pdm_docs/sd/532610271_sd.pdf), generated with kicad-footprint-generator")
+    (tags "connector Molex PicoBlade top entry")
+    (property "Sheetfile" "main_pcb.kicad_sch")
+    (property "Sheetname" "")
+    (attr smd)
+    (fp_text reference "J2" (at 0 -4.4) (layer "F.SilkS")
+      (effects (font (size 1 1) (thickness 0.15)))
+    )
+    (fp_text value "Conn_01x03" (at 0 3.8) (layer "F.Fab")
+      (effects (font (size 1 1) (thickness 0.15)))
+    )
+    (fp_text user "${REFERENCE}" (at 0 1.9) (layer "F.Fab")
+      (effects (font (size 1 1) (thickness 0.15)))
+    )
+    (fp_line (start -2.86 2.26) (end -2.86 2.71) (layer "F.SilkS") (width 0.12))
+    (fp_line (start -2.86 -1.71) (end -1.91 -1.71) (layer "F.SilkS") (width 0.12))
+    (fp_line (start 2.86 -1.26) (end 2.86 -1.71) (layer "F.SilkS") (width 0.12))
+    (fp_line (start -2.86 2.71) (end 2.86 2.71) (layer "F.SilkS") (width 0.12))
+    (fp_line (start -2.86 -1.26) (end -2.86 -1.71) (layer "F.SilkS") (width 0.12))
+    (fp_line (start 2.86 2.71) (end 2.86 2.26) (layer "F.SilkS") (width 0.12))
+    (fp_line (start -1.91 -1.71) (end -1.91 -3.2) (layer "F.SilkS") (width 0.12))
+    (fp_line (start 2.86 -1.71) (end 1.91 -1.71) (layer "F.SilkS") (width 0.12))
+    (fp_line (start -5.35 -3.7) (end -5.35 3.1) (layer "F.CrtYd") (width 0.05))
+    (fp_line (start 5.35 3.1) (end 5.35 -3.7) (layer "F.CrtYd") (width 0.05))
+    (fp_line (start -5.35 3.1) (end 5.35 3.1) (layer "F.CrtYd") (width 0.05))
+    (fp_line (start 5.35 -3.7) (end -5.35 -3.7) (layer "F.CrtYd") (width 0.05))
+    (fp_line (start -2.75 -0.6) (end -4.25 -0.6) (layer "F.Fab") (width 0.1))
+    (fp_line (start -4.25 -0.6) (end -4.45 -0.4) (layer "F.Fab") (width 0.1))
+    (fp_line (start 4.45 -0.4) (end 4.45 1.4) (layer "F.Fab") (width 0.1))
+    (fp_line (start -2.75 2.6) (end 2.75 2.6) (layer "F.Fab") (width 0.1))
+    (fp_line (start 4.25 2.2) (end 2.75 2.2) (layer "F.Fab") (width 0.1))
+    (fp_line (start 2.75 -0.6) (end 4.25 -0.6) (layer "F.Fab") (width 0.1))
+    (fp_line (start -4.45 1.4) (end -4.25 1.6) (layer "F.Fab") (width 0.1))
+    (fp_line (start -2.75 -1.6) (end -2.75 2.6) (layer "F.Fab") (width 0.1))
+    (fp_line (start -1.25 -0.892893) (end -0.75 -1.6) (layer "F.Fab") (width 0.1))
+    (fp_line (start -4.45 -0.4) (end -4.45 1.4) (layer "F.Fab") (width 0.1))
+    (fp_line (start 4.45 1.4) (end 4.25 1.6) (layer "F.Fab") (width 0.1))
+    (fp_line (start -4.25 1.6) (end -4.25 2.2) (layer "F.Fab") (width 0.1))
+    (fp_line (start -4.25 2.2) (end -2.75 2.2) (layer "F.Fab") (width 0.1))
+    (fp_line (start 4.25 1.6) (end 4.25 2.2) (layer "F.Fab") (width 0.1))
+    (fp_line (start 2.75 -1.6) (end 2.75 2.6) (layer "F.Fab") (width 0.1))
+    (fp_line (start -1.75 -1.6) (end -1.25 -0.892893) (layer "F.Fab") (width 0.1))
+    (fp_line (start 4.25 -0.6) (end 4.45 -0.4) (layer "F.Fab") (width 0.1))
+    (fp_line (start -2.75 -1.6) (end 2.75 -1.6) (layer "F.Fab") (width 0.1))
+    (pad "1" smd roundrect (at -1.25 -2.4) (size 0.8 1.6) (layers "F.Cu" "F.Paste" "F.Mask") (roundrect_rratio 0.25)
       (net 6 "+BATT") (pinfunction "Pin_1") (pintype "passive"))
-    (pad "2" thru_hole oval (at 2.5 0) (size 1.7 2) (drill 1) (layers *.Cu *.Mask)
-      (net 2 "GND") (pinfunction "Pin_2") (pintype "passive"))
-    (model "${KICAD6_3DMODEL_DIR}/Connector_JST.3dshapes/JST_XH_B2B-XH-AM_1x02_P2.50mm_Vertical.wrl"
-      (offset (xyz 0 0 0))
-      (scale (xyz 1 1 1))
+    (pad "2" smd roundrect (at 0 -2.4) (size 0.8 1.6) (layers "F.Cu" "F.Paste" "F.Mask") (roundrect_rratio 0.25)
+      (net 93 "unconnected-(J2-Pad2)") (pinfunction "Pin_2") (pintype "passive"))
+    (pad "3" smd roundrect (at 1.25 -2.4) (size 0.8 1.6) (layers "F.Cu" "F.Paste" "F.Mask") (roundrect_rratio 0.25)
+      (net 2 "GND") (pinfunction "Pin_3") (pintype "passive"))
+    (pad "MP" smd roundrect (at -3.8 0.5) (size 2.1 3) (layers "F.Cu" "F.Paste" "F.Mask") (roundrect_rratio 0.119048))
+    (pad "MP" smd roundrect (at 3.8 0.5) (size 2.1 3) (layers "F.Cu" "F.Paste" "F.Mask") (roundrect_rratio 0.119048))
+    (model "${KICAD6_3DMODEL_DIR}/Connector_Molex.3dshapes/Molex_PicoBlade_53261-0371_1x03-1MP_P1.25mm_Horizontal.wrl"
+      (offset (xyz 0 0 0))
+      (scale (xyz 1 1 1))

Commit message: Initial route
Parts:
- C4, C5, C7, C8: moved to B.Cu
- moved R9 123.8 mm to (39.2, 33.2), turned to 90 degrees
- moved C9 121.6 mm to (34.2, 62.8)
- moved R12 119.4 mm to (42.0, 35.8)
- moved C12 118.2 mm to (30.0, 56.5), turned to -90 degrees
- moved R11 117.7 mm to (42.0, 37.2), turned to 180 degrees
- moved C11 115.8 mm to (30.6, 53.2), turned to 180 degrees
- moved R13 114.1 mm to (31.5, 56.5), turned to -90 degrees
- moved Q3 113.1 mm to (42.0, 33.2)
- moved U3 112.4 mm to (34.8, 60.0)
- moved C15 110.8 mm to (41.0, 60.8), turned to 180 degrees
- moved R7 110.3 mm to (43.0, 67.8), turned to 180 degrees
- moved R14 109.4 mm to (31.5, 59.5), turned to -90 degrees
- moved R5 109.3 mm to (43.0, 69.2), turned to 180 degrees
- moved C13 109.0 mm to (33.5, 50.2), turned to 90 degrees
- moved R16 107.8 mm to (50.7, 39.3)
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Routing:
- net GND: track 0.00 -> 80.1 mm, vias 0 -> 13
- net +BATT: track 0.00 -> 44.1 mm
- net VBUS: track 0.00 -> 31.2 mm, vias 0 -> 3
- net +3.3V: track 0.00 -> 21.9 mm, vias 0 -> 6
- net D-: track 0.00 -> 20.1 mm, vias 0 -> 3
- net Net-(R6-Pad1): track 0.00 -> 18.8 mm
- net D+: track 0.00 -> 18.7 mm
- net +5V: track 0.00 -> 17.9 mm, vias 0 -> 3
- net Net-(J1-PadB5): track 0.00 -> 11.0 mm
- net Net-(Q1-Pad3): track 0.00 -> 10.0 mm
- net Net-(R16-Pad2): track 0.00 -> 9.16 mm
- net Net-(C14-Pad1): track 0.00 -> 8.98 mm
- net Net-(C3-Pad1): track 0.00 -> 8.67 mm
- net Net-(C10-Pad1): track 0.00 -> 8.63 mm
- net Net-(J6-Pad2): track 0.00 -> 6.84 mm
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- added copper zone on In2.Cu, net +3.3V
- added copper zone on B.Cu, net +5V
- added copper zone on In1.Cu, net GND

Commit message: Finished routing
Parts:
- moved R3 8.02 mm to (61.5, 58.9)
- moved C11 0.50 mm to (30.6, 53.8)
- moved C1 0.20 mm to (63.8, 52.7)
- turned D6 to -157.5 degrees
Connections:
- U4 pad 15: unconnected-(U4-Pad15) -> IO_OFF
- U4 pad 17: unconnected-(U4-Pad17) -> PUSH_UP
- U4 pad 18: unconnected-(U4-Pad18) -> PUSH
- U4 pad 20: unconnected-(U4-Pad20) -> MOTOR_UH
- U4 pad 21: unconnected-(U4-Pad21) -> MOTOR_UL
- U4 pad 22: unconnected-(U4-Pad22) -> MOTOR_VH
- U4 pad 23: unconnected-(U4-Pad23) -> MOTOR_VL
- U4 pad 24: unconnected-(U4-Pad24) -> MOTOR_WH
- U4 pad 25: unconnected-(U4-Pad25) -> MOTOR_WL
- U4 pad 28: unconnected-(U4-Pad28) -> MOTOR_DIAG
- U4 pad 29: unconnected-(U4-Pad29) -> MM_SDA
- U4 pad 30: unconnected-(U4-Pad30) -> MM_SCL
- U4 pad 31: unconnected-(U4-Pad31) -> MM_CS
- U4 pad 32: unconnected-(U4-Pad32) -> LCD_BL
- U4 pad 33: unconnected-(U4-Pad33) -> LCD_DC
- U4 pad 34: unconnected-(U4-Pad34) -> LCD_CS
- U4 pad 35: unconnected-(U4-Pad35) -> LCD_SCL
- U4 pad 38: unconnected-(U4-Pad38) -> LCD_SDA
- U4 pad 39: unconnected-(U4-Pad39) -> LCD_RESET
- U4 pad 4: unconnected-(U4-Pad4) -> RGB
- U4 pad 5: unconnected-(U4-Pad5) -> BAT_ADC
- U4 pad 6: unconnected-(U4-Pad6) -> BAT_ADC_EN
Routing:
- net BAT_ADC_EN: track 0.00 -> 35.8 mm, vias 0 -> 2
- net GND: track 80.1 -> 111.5 mm, vias 13 -> 25
- net BAT_ADC: track 1.50 -> 29.0 mm, vias 0 -> 2
- net PUSH: track 1.76 -> 26.7 mm, vias 0 -> 3
- net Net-(D4-Pad3): track 0.00 -> 18.9 mm, vias 0 -> 2
- net Net-(D4-Pad1): track 0.00 -> 16.2 mm, vias 0 -> 2
- net Net-(D3-Pad1): track 0.00 -> 13.7 mm, vias 0 -> 2
- net Net-(D1-Pad1): track 0.00 -> 13.3 mm, vias 0 -> 2
- net Net-(D2-Pad1): track 0.00 -> 13.3 mm, vias 0 -> 2
- net Net-(D2-Pad3): track 0.00 -> 13.2 mm, vias 0 -> 2
- net LCD_BL: track 0.00 -> 13.1 mm, vias 0 -> 1
- net Net-(D3-Pad3): track 0.00 -> 13.0 mm
- net LCD_DC: track 0.00 -> 11.7 mm, vias 0 -> 1
- net MOTOR_UH: track 0.00 -> 11.6 mm, vias 0 -> 1
- net LCD_CS: track 0.00 -> 10.3 mm, vias 0 -> 1
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