File: hardware/lcd_pcb/lcd_pcb.kicad_sch (KiCad schematic)
At the start: 7 parts

Commit message: Added footprint for lcd
Parts:
- J?: footprint (none) -> LCD_GC9A01:GC9A01Round1.28
Changed lines of the file:
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@@
     (property "Reference" "J?" (id 0) (at 116.84 73.66 0))
     (property "Value" "LCD" (id 1) (at 116.84 76.2 0))
-    (property "Footprint" "" (id 2) (at 116.84 92.71 0)
+    (property "Footprint" "LCD_GC9A01:GC9A01Round1.28" (id 2) (at 116.84 92.71 0)
       (effects (font (size 1.27 1.27)) hide)
     )
@@
     )
     (path "/bbf0e25e-ecad-4bfd-80c9-1fb75474b3d9"
-      (reference "J?") (unit 1) (value "LCD") (footprint "")
+      (reference "J?") (unit 1) (value "LCD") (footprint "LCD_GC9A01:GC9A01Round1.28")
     )
     (path "/f6777b3f-7832-45d1-bf4b-ad0fde6a7abd"

Commit message: Designed lcd pcb
Parts:
- gave numbers to parts that had none: 7
Changed lines of the file:
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@@
   (symbol (lib_id "power:GND") (at 128.27 118.11 0) (unit 1)
     (in_bom yes) (on_board yes) (fields_autoplaced)
-    (property "Reference" "#PWR?" (id 0) (at 128.27 124.46 0)
+    (property "Reference" "#PWR0102" (id 0) (at 128.27 124.46 0)
       (effects (font (size 1.27 1.27)) hide)
     )
@@
   (symbol (lib_id "Device:R") (at 140.97 82.55 90) (unit 1)
     (in_bom yes) (on_board yes) (fields_autoplaced)
-    (property "Reference" "R?" (id 0) (at 140.97 76.2 90))
+    (property "Reference" "R1" (id 0) (at 140.97 76.2 90))
     (property "Value" "10" (id 1) (at 140.97 78.74 90))
     (property "Footprint" "Resistor_SMD:R_0603_1608Metric" (id 2) (at 140.97 84.328 90)
@@
   (symbol (lib_id "power:GND") (at 175.26 100.33 0) (unit 1)
     (in_bom yes) (on_board yes) (fields_autoplaced)
-    (property "Reference" "#PWR?" (id 0) (at 175.26 106.68 0)
+    (property "Reference" "#PWR0101" (id 0) (at 175.26 106.68 0)
       (effects (font (size 1.27 1.27)) hide)
     )
@@
   (symbol (lib_id "Connector_Generic:Conn_01x08") (at 182.88 87.63 0) (unit 1)
     (in_bom yes) (on_board yes) (fields_autoplaced)
-    (property "Reference" "J?" (id 0) (at 185.42 87.6299 0)
+    (property "Reference" "J2" (id 0) (at 185.42 87.6299 0)
       (effects (font (size 1.27 1.27)) (justify left))
     )
@@
   (symbol (lib_id "Device:C") (at 134.62 111.76 0) (unit 1)
     (in_bom yes) (on_board yes) (fields_autoplaced)
-    (property "Reference" "C?" (id 0) (at 138.43 110.4899 0)
+    (property "Reference" "C1" (id 0) (at 138.43 110.4899 0)
       (effects (font (size 1.27 1.27)) (justify left))
     )
@@
   (symbol (lib_id "power:+3.3V") (at 134.62 76.2 0) (unit 1)
     (in_bom yes) (on_board yes) (fields_autoplaced)
-    (property "Reference" "#PWR?" (id 0) (at 134.62 80.01 0)
+    (property "Reference" "#PWR0103" (id 0) (at 134.62 80.01 0)
       (effects (font (size 1.27 1.27)) hide)
     )
@@
   (symbol (lib_id "Connector_Generic:Conn_01x12") (at 116.84 92.71 0) (mirror y) (unit 1)
     (in_bom yes) (on_board yes) (fields_autoplaced)
-    (property "Reference" "J?" (id 0) (at 116.84 73.66 0))
+    (property "Reference" "J1" (id 0) (at 116.84 73.66 0))
     (property "Value" "LCD" (id 1) (at 116.84 76.2 0))
     (property "Footprint" "LCD_GC9A01:GC9A01Round1.28" (id 2) (at 116.84 92.71 0)
@@
   (symbol (lib_id "Device:R") (at 161.29 82.55 90) (unit 1)
     (in_bom yes) (on_board yes) (fields_autoplaced)
-    (property "Reference" "R?" (id 0) (at 161.29 76.2 90))
+    (property "Reference" "R3" (id 0) (at 161.29 76.2 90))
     (property "Value" "10" (id 1) (at 161.29 78.74 90))
     (property "Footprint" "Resistor_SMD:R_0603_1608Metric" (id 2) (at 161.29 84.328 90)
@@
   (symbol (lib_id "Transistor_FET:AO3400A") (at 149.86 87.63 0) (mirror y) (unit 1)
     (in_bom yes) (on_board yes)
-    (property "Reference" "Q?" (id 0) (at 143.51 86.3599 0)
+    (property "Reference" "Q1" (id 0) (at 143.51 86.3599 0)
       (effects (font (size 1.27 1.27)) (justify left))
     )
@@
   (symbol (lib_id "Device:R") (at 156.21 111.76 180) (unit 1)
     (in_bom yes) (on_board yes) (fields_autoplaced)
-    (property "Reference" "R?" (id 0) (at 158.75 110.4899 0)
+    (property "Reference" "R2" (id 0) (at 158.75 110.4899 0)
       (effects (font (size 1.27 1.27)) (justify right))
     )
@@
   )
   (symbol_instances
+    (path "/5e30750f-dbb3-4f45-b648-968fe8864f1a"
+      (reference "#PWR0101") (unit 1) (value "GND") (footprint "")
+    )
     (path "/25062e09-860e-44cc-abde-a01971751c92"
-      (reference "#PWR?") (unit 1) (value "GND") (footprint "")
-    )
-    (path "/5e30750f-dbb3-4f45-b648-968fe8864f1a"
-      (reference "#PWR?") (unit 1) (value "GND") (footprint "")
+      (reference "#PWR0102") (unit 1) (value "GND") (footprint "")
     )
     (path "/b9083343-779f-4c80-bab8-875871514b42"
-      (reference "#PWR?") (unit 1) (value "+3.3V") (footprint "")
+      (reference "#PWR0103") (unit 1) (value "+3.3V") (footprint "")
     )
     (path "/b2ea4103-0bb1-4f1f-91ee-2697186646ac"
-      (reference "C?") (unit 1) (value "100nF") (footprint "Capacitor_SMD:C_0603_1608Metric")
+      (reference "C1") (unit 1) (value "100nF") (footprint "Capacitor_SMD:C_0603_1608Metric")
+    )
+    (path "/bbf0e25e-ecad-4bfd-80c9-1fb75474b3d9"
+      (reference "J1") (unit 1) (value "LCD") (footprint "LCD_GC9A01:GC9A01Round1.28")
     )
     (path "/9a881769-4e23-4dd3-b882-f6a948996f5a"
-      (reference "J?") (unit 1) (value "main") (footprint "Connector_Hirose:Hirose_DF52-8S-0.8H_1x08-1MP_P0.80mm_Horizontal")
-    )
-    (path "/bbf0e25e-ecad-4bfd-80c9-1fb75474b3d9"
-      (reference "J?") (unit 1) (value "LCD") (footprint "LCD_GC9A01:GC9A01Round1.28")
+      (reference "J2") (unit 1) (value "main") (footprint "Connector_Hirose:Hirose_DF52-8S-0.8H_1x08-1MP_P0.80mm_Horizontal")
     )
     (path "/f6777b3f-7832-45d1-bf4b-ad0fde6a7abd"
-      (reference "Q?") (unit 1) (value "AO3400A") (footprint "Package_TO_SOT_SMD:SOT-23")
+      (reference "Q1") (unit 1) (value "AO3400A") (footprint "Package_TO_SOT_SMD:SOT-23")
     )
     (path "/57004d4f-90c5-4ddf-b2d6-f6d2211ced01"
-      (reference "R?") (unit 1) (value "10") (footprint "Resistor_SMD:R_0603_1608Metric")
+      (reference "R1") (unit 1) (value "10") (footprint "Resistor_SMD:R_0603_1608Metric")
+    )
+    (path "/fbe2ab5e-d28e-4670-af06-3a1407c43d9a"
+      (reference "R2") (unit 1) (value "10k") (footprint "Resistor_SMD:R_0603_1608Metric")
     )
     (path "/cc9bd8a8-b257-4091-991d-979ba4d74ee3"
-      (reference "R?") (unit 1) (value "10") (footprint "Resistor_SMD:R_0603_1608Metric")
-    )
-    (path "/fbe2ab5e-d28e-4670-af06-3a1407c43d9a"
-      (reference "R?") (unit 1) (value "10k") (footprint "Resistor_SMD:R_0603_1608Metric")
-    )
-  )
+      (reference "R3") (unit 1) (value "10") (footprint "Resistor_SMD:R_0603_1608Metric")
+    )
+  )

Commit message: Use spi
Parts:
- J2: LCSC (none) -> C500143
Changed lines of the file:
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@@
+      (effects (font (size 1.27 1.27)) hide)
+    )
+    (property "LCSC" "C500143" (id 4) (at 182.88 87.63 0)
       (effects (font (size 1.27 1.27)) hide)
     )
